File: rat-ratgdo esphome sensor/rat-ratgdo esphome sensor.kicad_pcb (KiCad board)
At the start: 2 copper layers, 45.7 x 42.9 mm, 34 parts, among them J1 Analog in, J2 Conn_02x03_Odd_Even, J3 UJ2-MIBH-G-SMT-TR, J4 LUX sensor, J6 bme280, J7 qwiic, J8 power, J9 GDO, Q1 2N7002, Q2 AO3400A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

Commit message: revisions for design error
Routing:
- net GND: track 2.54 -> 64.8 mm, vias 0 -> 2
Changed lines of the file:
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@@
   (segment (start 77.52 36.893) (end 77.47 36.843) (width 0.6) (layer "F.Cu") (net 1))
   (segment (start 102.371767 36.81) (end 103.124 36.057767) (width 0.4) (layer "F.Cu") (net 1))
+  (segment (start 108.458 55.372) (end 109.0445 54.7855) (width 0.6) (layer "F.Cu") (net 2))
+  (segment (start 89.877 54.659) (end 90.322 55.104) (width 1) (layer "F.Cu") (net 2))
+  (segment (start 102.235 49.53) (end 101.028 50.737) (width 0.6) (layer "F.Cu") (net 2))
+  (segment (start 103.569 45.784) (end 103.633 45.72) (width 0.6) (layer "F.Cu") (net 2))
+  (segment (start 96.012 61.722) (end 97.282 62.992) (width 0.4) (layer "F.Cu") (net 2))
+  (segment (start 99.0345 50.8555) (end 99.06 50.83) (width 0.6) (layer "F.Cu") (net 2))
+  (segment (start 87.884 54.659) (end 89.877 54.659) (width 1) (layer "F.Cu") (net 2))
+  (segment (start 78.994 38.228) (end 75.693 38.228) (width 0.4) (layer "F.Cu") (net 2))
+  (segment (start 91.923 63.525) (end 91.923 66.1) (width 0.4) (layer "F.Cu") (net 2))
+  (segment (start 100.393 50.737) (end 100.3 50.83) (width 0.6) (layer "F.Cu") (net 2))
+  (segment (start 90.322 55.104) (end 94.121 55.104) (width 1) (layer "F.Cu") (net 2))
+  (segment (start 100.3 50.83) (end 99.06 50.83) (width 0.6) (layer "F.Cu") (net 2))
+  (segment (start 104.297 55.372) (end 108.458 55.372) (width 0.6) (layer "F.Cu") (net 2))
+  (segment (start 96.48 52.745) (end 96.48 52.07) (width 1) (layer "F.Cu") (net 2))
+  (segment (start 75.565 38.1) (end 75.565 35.56) (width 0.4) (layer "F.Cu") (net 2))
+  (segment (start 96.734 52.324) (end 96.48 52.07) (width 0.6) (layer "F.Cu") (net 2))
+  (segment (start 75.693 38.228) (end 75.565 38.1) (width 0.4) (layer "F.Cu") (net 2))
+  (segment (start 105.786 49.53) (end 102.235 49.53) (width 0.6) (layer "F.Cu") (net 2))
+  (segment (start 75.832 35.293) (end 77.47 35.293) (width 0.4) (layer "F.Cu") (net 2))
+  (segment (start 94.121 55.104) (end 96.48 52.745) (width 1) (layer "F.Cu") (net 2))
+  (segment (start 102.4405 55.435) (end 104.234 55.435) (width 0.6) (layer "F.Cu") (net 2))
+  (segment (start 104.234 55.435) (end 104.297 55.372) (width 0.6) (layer "F.Cu") (net 2))
   (segment (start 73.914 58.674) (end 71.374 58.674) (width 0.4) (layer "F.Cu") (net 2))
+  (segment (start 99.0345 52.324) (end 96.734 52.324) (width 0.6) (layer "F.Cu") (net 2))
+  (segment (start 101.028 50.737) (end 100.393 50.737) (width 0.6) (layer "F.Cu") (net 2))
+  (segment (start 91.948 63.5) (end 91.948 61.722) (width 0.4) (layer "F.Cu") (net 2))
+  (segment (start 91.948 61.722) (end 96.012 61.722) (width 0.4) (layer "F.Cu") (net 2))
+  (segment (start 99.06 50.83) (end 96.48 50.83) (width 0.6) (layer "F.Cu") (net 2))
+  (segment (start 97.282 62.992) (end 99.822 62.992) (width 0.4) (layer "F.Cu") (net 2))
+  (segment (start 100.393 48.768) (end 100.393 50.737) (width 0.6) (layer "F.Cu") (net 2))
+  (segment (start 103.633 45.72) (end 107.95 45.72) (width 0.6) (layer "F.Cu") (net 2))
+  (segment (start 96.48 52.07) (end 96.48 50.83) (width 1) (layer "F.Cu") (net 2))
+  (segment (start 109.0445 54.7855) (end 109.0445 53.914) (width 0.6) (layer "F.Cu") (net 2))
+  (segment (start 103.569 46.736) (end 103.569 45.784) (width 0.6) (layer "F.Cu") (net 2))
+  (segment (start 99.0345 52.324) (end 99.0345 50.8555) (width 0.6) (layer "F.Cu") (net 2))
+  (segment (start 106.172 49.916) (end 105.786 49.53) (width 0.6) (layer "F.Cu") (net 2))
+  (segment (start 75.565 35.56) (end 75.832 35.293) (width 0.4) (layer "F.Cu") (net 2))
+  (segment (start 91.923 66.1) (end 91.848 66.175) (width 0.4) (layer "F.Cu") (net 2))
+  (segment (start 91.948 63.5) (end 91.923 63.525) (width 0.4) (layer "F.Cu") (net 2))
+  (via (at 85.725 61.595) (size 0.8) (drill 0.4) (layers "F.Cu" "B.Cu") (free) (net 2))
+  (via (at 85.725 54.61) (size 0.8) (drill 0.4) (layers "F.Cu" "B.Cu") (free) (net 2))
   (segment (start 104.889 33.515) (end 104.394 33.02) (width 0.6) (layer "F.Cu") (net 3))
   (segment (start 89.348 63.5) (end 89.348 60.678) (width 0.4) (layer "F.Cu") (net 3))
@@
   (via (at 103.886 43.18) (size 0.8) (drill 0.4) (layers "F.Cu" "B.Cu") (net 13))
   (segment (start 103.886 50.8) (end 103.886 43.18) (width 0.4) (layer "B.Cu") (net 13))
-  (segment (start 103.984 53.785) (end 104.297 53.472) (width 0.6) (layer "F.Cu") (net 14))
   (segment (start 102.4405 53.785) (end 102.362 53.594) (width 0.6) (layer "F.Cu") (net 14))
   (segment (start 102.362 40.894) (end 102.298 40.83) (width 0.4) (layer "F.Cu") (net 14))
-  (segment (start 102.362 53.594) (end 103.984 53.785) (width 0.6) (layer "F.Cu") (net 14))
+  (segment (start 104.175 53.594) (end 104.297 53.472) (width 0.6) (layer "F.Cu") (net 14))
+  (segment (start 102.362 53.594) (end 104.175 53.594) (width 0.6) (layer "F.Cu") (net 14))
   (segment (start 102.298 40.83) (end 96.48 40.83) (width 0.4) (layer "F.Cu") (net 14))
   (via (at 102.362 53.594) (size 0.8) (drill 0.4) (layers "F.Cu" "B.Cu") (net 14))
@@
     (connect_pads (clearance 0))
     (min_thickness 0.25) (filled_areas_thickness no)
-    (keepout (tracks allowed) (vias not_allowed) (pads not_allowed) (copperpour not_allowed) (footprints allowed))
+    (keepout (tracks allowed) (vias allowed) (pads allowed) (copperpour not_allowed) (footprints allowed))
     (fill (thermal_gap 0.5) (thermal_bridge_width 0.5))
     (polygon
